File: memory_controller.sch (KiCad schematic (older format))
At the start: 38 parts, among them SW1 SW_DIP_x03, U14 STM32F407VGTx

Commit message: New layout and design
Parts:
- removed R23: 0, Resistors_SMD:R_1206_HandSoldering, symbol R_Small
- removed U14: STM32F407VGTx, Housings_QFP:TQFP-100_14x14mm_Pitch0.5mm, symbol STM32F407VGTx
- added C18, C19, C20, C21, C22, C23, C24, C25: 100n, Capacitors_SMD:C_1206_HandSoldering, symbol C_Small
- added C9: 1u, Capacitors_SMD:C_1206_HandSoldering, symbol C_Small
- added U3: STM32F407IGTx, Housings_QFP:LQFP-176_24x24mm_Pitch0.5mm, symbol STM32F407IGTx
- C10: renamed from C32; value 1u -> 100n
- renumbered C21 to C11, C22 to C12, C23 to C13, C24 to C14, C25 to C15, C26 to C16, C27 to C17, C33 to C4, C34 to C5, C19 to C6, C20 to C7, C31 to C8, D5 to D1, R19 to R10, R26 to R11, R27 to R12, R30 to R13, R20 to R14, R28 to R15, R29 to R16, R21 to R17, R31 to R18, R32 to R19, R24 to R20, R2 to R3, R3 to R4, R4 to R5, R5 to R6, R18 to R9, SW1 to SW2, XT2 to XT1
Connections:
- net GND: now also C18.1, C19.1, C20.1, C21.1, C22.1, C23.1, C24.1, C25.1, C9.1, U3.102 (VSS), U3.113 (VSS), U3.126 (VSS), U3.135 (VSS), U3.14 (VSS), U3.148 (VSS), U3.158 (VSS), U3.22 (VSS), U3.61 (VSS), U3.71 (VSS), U3.90 (VSS); no longer R14.1, R17.1
- net LEDGRN_MEM: now also U3.56 (PB0)
- net PB6: now also U3.164 (PB6)
- net PB9: now also U3.168 (PB9)
- net SWDCLK_MEM: now also U3.137 (PA14)
- net SWDIO_MEM: now also U3.124 (PA13)
- net UART_RX: now also U3.121 (PA10)
- net UART_TX: now also U3.120 (PA9)
- net VCAP_1_MEM: now also U3.81 (VCAP_1)
- net VCAP_2_MEM: now also U3.125 (VCAP_2)
- net VCC_3V3: now also R14.1, R17.1, C18.2, C19.2, C20.2, C21.2, C22.2, C23.2, C24.2, C25.2, U3.103 (VDD), U3.114 (VDD), U3.127 (VDD), U3.136 (VDD), U3.149 (VDD), U3.15 (VDD), U3.159 (VDD), U3.172 (VDD), U3.23 (VDD), U3.36 (VDD), U3.38 (VREF+), U3.39 (VDDA), U3.49 (VDD), U3.62 (VDD), U3.72 (VDD), U3.82 (VDD), U3.91 (VDD)
- net mA0: now also U3.32 (PC0)
- net mA1: now also U3.33 (PC1)
- net mA10: now also U3.139 (PC10)
- net mA11: now also U3.140 (PC11)
- net mA12: now also U3.141 (PC12)
- net mA13: now also U3.8 (PC13)
- net mA14: now also U3.9 (PC14)
- net mA15: now also U3.10 (PC15)
- net mA2: now also U3.34 (PC2)
- net mA3: now also U3.35 (PC3)
- net mA4: now also U3.54 (PC4)
- net mA5: now also U3.55 (PC5)
- net mA6: now also U3.115 (PC6)
- net mA7: now also U3.116 (PC7)
- net mA8: now also U3.117 (PC8)
- net mA9: now also U3.118 (PC9)
- net mCONF0: now also U3.7 (PI8)
- net mCONF1: now also U3.176 (PI7)
- net mCONF2: now also U3.175 (PI6)
- net mD0: now also U3.40 (PA0)
- net mD1: now also U3.41 (PA1)
- net mD2: now also U3.42 (PA2)
- net mD3: now also U3.47 (PA3)
- net mD4: now also U3.50 (PA4)
- net mD5: now also U3.51 (PA5)
- net mD6: now also U3.52 (PA6)
- net mD7: now also U3.53 (PA7)
- net mPHI2: now also U3.131 (PI0)
- net mR/~W: now also U3.174 (PI5)
- net mRD4: now also U3.162 (PB4)
- net mRD5: now also U3.58 (PB2)
- net nRESET_MEM: now also U3.31 (NRST)
- net ~mCCTL: now also U3.173 (PI4)
- net ~mD1XX: now also U3.134 (PI3)
- net ~mEXSEL: now also U3.163 (PB5)
- net ~mHALT: now also U3.165 (PB7)
- net ~mIRQ: now also U3.79 (PB10)
- net ~mMPD: now also U3.167 (PB8)
- net ~mREF: now also U3.161 (PB3)
- net ~mRST: now also U3.57 (PB1)
- net ~mS4: now also U3.133 (PI2)
- net ~mS5: now also U3.132 (PI1)
- net at R10.1: now also U3.30 (PH1)
- net at R9.1: now also U3.29 (PH0)
- net at R13.1: now also U3.37 (VSSA)
- net at R11.2, R12.1: now also U3.166 (BOOT0)
- new net: C9.2, U3.6 (VBAT)
- new net FSMC_A0: U3.16 (PF0)
- new net FSMC_A1: U3.17 (PF1)
- new net FSMC_A10: U3.66 (PG0)
- new net FSMC_A11: U3.67 (PG1)
- new net FSMC_A12: U3.106 (PG2)
- new net FSMC_A13: U3.107 (PG3)
- new net FSMC_A14: U3.108 (PG4)
- new net FSMC_A15: U3.109 (PG5)
- new net FSMC_A16: U3.99 (PD11)
- new net FSMC_A17: U3.100 (PD12)
- new net FSMC_A18: U3.101 (PD13)
- new net FSMC_A2: U3.18 (PF2)
- new net FSMC_A3: U3.19 (PF3)
- new net FSMC_A4: U3.20 (PF4)
- new net FSMC_A5: U3.21 (PF5)
- new net FSMC_A6: U3.60 (PF12)
- new net FSMC_A7: U3.63 (PF13)
- new net FSMC_A8: U3.64 (PF14)
- new net FSMC_A9: U3.65 (PF15)
- new net FSMC_D0: U3.104 (PD14)
- new net FSMC_D1: U3.105 (PD15)
- new net FSMC_D2: U3.142 (PD0)
- new net FSMC_D3: U3.143 (PD1)
- new net FSMC_D4: U3.68 (PE7)
- new net FSMC_D5: U3.69 (PE8)
- new net FSMC_D6: U3.70 (PE9)
- new net FSMC_D7: U3.73 (PE10)
- new net FSMC_NE1: U3.151 (PD7)
- new net FSMC_NE2: U3.152 (PG9)
- new net FSMC_NOE: U3.146 (PD4)
- new net FSMC_NWE: U3.147 (PD5)
- no-connect marks 21 -> 61
Other:
- note removed: "130XE the internal extra 64K RAM are disabled by default. Only External RAM is available."
- note removed: "64 of 16K banks addressable (TOTAL 1024K)"
- note removed: "TEST RAM UP TO 1.5MB"
- moved on the sheet: BOOT0_MEM1, BOOT1_MEM1, C10, C11, C12, C13, C14, C15, C16, C17, C4, C5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
